File: board/mmp.sch (KiCad schematic (older format))
At the start: 66 parts, among them IC1 STM32F103C, IC2 SI8662, IC3 SI8662, IC4 MCP1700-33, IC5 MCP1700-33, IC6 TXS0108, IC7 1117-SOT223, J1 SWD, P1 USB_B, P2 CONN_01X04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

Commit message: finishing off
Parts:
- R1, R10, R11, R12, R13, R14, R15, R16, R17, R18, R19, R2, R20, R21, R22, R3, R4, R5, R6, R7, R8, R9: footprint Resistors_SMD:R_0603 -> passives-7351:C0603-N
- SW1, SW3: footprint Buttons_Switches_SMD:SW_SPST_EVQPE1 -> tactile_SPST:SW_SPST_EVQPE1
- Y1: footprint Crystals:Crystal_FOX-FE_SMD -> ABM7:ABM7

Commit message: done
Parts:
- P2: footprint Connectors_Molex:Connector_Molex_PicoBlade_53261-0471 -> agg:SM04B-PASS
Connections:
- wire segments 238 -> 239
Changed lines of the file:
@@
 F 0 "P2" H 10800 1050 50  0000 C CNN
 F 1 "CONN_01X04" V 10900 800 50  0000 C CNN
-F 2 "Connectors_Molex:Connector_Molex_PicoBlade_53261-0471" H 10800 800 60  0001 C CNN
+F 2 "agg:SM04B-PASS" H 10800 800 60  0001 C CNN
 F 3 "" H 10800 800 60  0000 C CNN
 	1    10800 800
@@
 	4600 3250 4350 3250
 Wire Wire Line
-	4900 3250 4900 3450
-Wire Wire Line
 	4100 3450 4800 3450
 Wire Wire Line
@@
 	7850 1400 7850 1600
 Connection ~ 7850 1600
+Wire Wire Line
+	5100 2850 5100 3450
+Wire Wire Line
+	5100 3450 4900 3450
 $EndSCHEMATC
