File: board-mini/mmp.kicad_pcb (KiCad board)
At the start: 2 copper layers, 50 x 15.2 mm, 39 parts, among them IC1 STM32F103C, IC3 SI8662, IC4 MCP1700-33, J1 SWD, P1 USB_B, P2 CONN_01X04, SW1 SW_PUSH, SW3 SW_PUSH, Y1 Crystal_Small

Commit message: finishing off
Parts:
- R1, R10, R11, R12, R13, R15, R2, R3, R4, R5, R6, R7, R8, R9: footprint Resistors_SMD:R_0603 -> passives-7351:C0603-N
- SW1, SW3: footprint Buttons_Switches_SMD:SW_SPST_EVQPE1 -> tactile_SPST:SW_SPST_EVQPE1
- Y1: footprint Crystals:Crystal_FOX-FE_SMD -> ABM7:ABM7
- moved SW1 0.76 mm to (214.1, 89.0)
- moved D4 0.60 mm to (204.4, 77.7)
- moved R11 0.60 mm to (204.4, 80.3)
- moved SW3 0.38 mm to (182.8, 89.1)
- moved D3 0.32 mm to (205.9, 77.7)
- moved R10 0.32 mm to (205.9, 80.3)
- moved R9 0.13 mm to (209.0, 80.3)
- moved D2 0.13 mm to (209.0, 77.7)
Routing:
- net +3V3: track 79.4 -> 77.9 mm
- net /SWDIO: track 25.2 -> 23.9 mm

Commit message: finishing off
Parts:
- moved C3 6.66 mm to (205.2, 83.1), turned to 180 degrees
- moved C1 1.02 mm to (208.0, 87.4)
- moved C4 1.02 mm to (208.0, 84.5)
- moved Y1 0.89 mm to (205.3, 87.4)
- moved R15 0.80 mm to (196.5, 89.5)
- moved C5 0.68 mm to (199.6, 89.5)
- moved R1 0.63 mm to (190.1, 77.9)
- moved R4 0.52 mm to (190.1, 85.7)
- moved R6 0.51 mm to (190.1, 79.6)
- moved C19 0.40 mm to (221.8, 77.7), turned to 270 degrees
- moved R13 0.36 mm to (222.1, 83.9)
- moved R3 0.25 mm to (190.1, 84.1)
- moved R5 0.25 mm to (190.1, 81.1)
- moved R7 0.25 mm to (222.2, 88.5)
- moved C9 0.13 mm to (191.2, 89.2)
Routing:
- net /SWDIO: track 23.9 -> 27.2 mm
- net GND: track 45.0 -> 48.2 mm, vias 18 -> 17
- net /Rx: track 11.4 -> 9.14 mm
- net GNDREF: track 27.5 -> 28.9 mm, vias 3 -> 2
- net Net-(IC1-Pad25): track 36.9 -> 35.7 mm
- net +3V3: track 77.9 -> 78.9 mm
- net Net-(IC3-Pad15): track 12.3 -> 11.3 mm
- net Net-(C4-Pad1): track 7.11 -> 7.96 mm
- net /H_SWCLK: track 33.2 -> 34.0 mm
- net Net-(IC1-Pad33): track 3.70 -> 3.00 mm
- net Net-(C1-Pad1): track 11.9 -> 11.4 mm
- net (no net): track 0.52 -> 0.00 mm
- net +3.3VP: track 20.0 -> 20.5 mm

Commit message: done
Parts:
- J1: footprint Pin_Headers:Pin_Header_Straight_2x05_Pitch1.27mm -> agg:FTSH-105-01-L-DV-K
- P2: footprint Connectors_Molex:Connector_Molex_PicoBlade_53261-0471 -> agg:SM04B-PASS
- moved D5 47.1 mm to (208.6, 44.4), turned to 90 degrees
- moved J1 46.7 mm to (203.5, 45.2)
- moved R14 42.9 mm to (210.1, 47.3), turned to 270 degrees
- moved R13 39.1 mm to (208.5, 47.2), turned to 90 degrees
- moved C11 38.4 mm to (197.8, 47.7), turned to 0 degrees
- moved SW2 33.9 mm to (209.1, 55.4), turned to 270 degrees
- moved P2 33.7 mm to (203.4, 49.5), turned to 180 degrees
- moved IC3 32.1 mm to (201.5, 53.1), turned to 0 degrees
- moved R12 26.8 mm to (203.5, 57.8), turned to 0 degrees
- moved SW1 26.5 mm to (209.2, 86.7), turned to 270 degrees
- moved C1 25.9 mm to (207.6, 61.5), turned to 180 degrees
- moved C7 25.3 mm to (210.1, 83.9), turned to 90 degrees
- moved C10 24.2 mm to (197.8, 57.8), turned to 0 degrees
- moved Y1 23.4 mm to (207.6, 64.2), turned to 180 degrees
- moved C4 23.2 mm to (204.7, 61.5), turned to 0 degrees
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- renumbered C18 to C10, C19 to C11, IC4 to IC2, R5 to R1, R15 to R10, R7 to R14, R8 to R2, R9 to R3, R10 to R4, R6 to R5, R1 to R6, R2 to R7, R3 to R8, R4 to R9, SW3 to SW1, SW1 to SW2
Connections:
- P1 pad 4: GND -> Net-(P1-Pad4)
- P1 pad 5: Net-(P1-Pad5) -> GND
Routing:
- net +3.3VP: track 20.5 -> 33.6 mm, vias 1 -> 2
- net GNDREF: track 28.9 -> 20.4 mm, vias 2 -> 3
- net Net-(IC3-Pad12): track 2.28 -> 9.85 mm
- net /Rx: track 9.14 -> 3.24 mm
- net /Tx: track 4.24 -> 7.94 mm
- net Net-(IC3-Pad14): track 5.66 -> 2.88 mm
- net Net-(IC3-Pad11): track 6.41 -> 7.63 mm
- net Net-(D5-Pad1): track 1.19 -> 2.26 mm
- net GND: track 48.2 -> 49.2 mm
- net /H_SWDIO: track 34.8 -> 35.4 mm
Other:
- board size 50 x 15.2 mm -> 15.2 x 50 mm
- board text added: "Feb 2016"
- board text added: "MMP-Isolated"
