File: board-mini/mmp.sch (KiCad schematic (older format))
At the start: 66 parts, among them IC1 STM32F103C, IC2 SI8662, IC3 SI8662, IC4 MCP1700-33, IC5 MCP1700-33, IC6 TXS0108, IC7 1117-SOT223, J1 SWD, P1 USB_B, P2 CONN_01X04, P3 TC2030-CTX, Q1 2n2007, Q2 NTR4101, SW1 SW_PUSH, SW2 SP3T, SW3 SW_PUSH, U2 ROE-0505S, Y1 Crystal_Small

Commit message: mostly done
Parts:
- removed C10, C12: 100n, Capacitors_SMD:C_0603, symbol C_Small
- removed C11, C13, C14: 4.7u, Capacitors_SMD:C_0603, symbol C_Small
- removed C15, C17: 10u, Capacitors_SMD:C_0805, symbol C_Small
- removed C16: 470p 4kV, symbol C_Small
- removed D6: LED, LEDs:LED-0603, symbol LED
- removed IC2: SI8662, SMD_Packages:SO-16-N, symbol SI8662
- removed IC5: MCP1700-33, TO_SOT_Packages_SMD:SOT-23, symbol reg-sot23
- removed IC6: TXS0108, Housings_SSOP:TSSOP-20_4.4x6.5mm_Pitch0.65mm, symbol TXS0108
- removed IC7: 1117-SOT223, TO_SOT_Packages_SMD:SOT-223, symbol 1117-SOT223
- removed L1: 4.7u, Inductors_NEOSID:Neosid_Inductor_SM-NE30_SMD1210, symbol L_Small
- removed Q1: 2n2007, TO_SOT_Packages_SMD:SOT-23, symbol Q_NMOS_GSD
- removed Q2: NTR4101, TO_SOT_Packages_SMD:SOT-23, symbol Q_PMOS_DGS
- removed R14, R16, R17, R18: 4.7k, Resistors_SMD:R_0603, symbol R_Small
- removed R19: 10k, Resistors_SMD:R_0603, symbol R_Small
- removed R20: 330, Resistors_SMD:R_0603, symbol R_Small
- removed SW2: SP3T, slide_SP3T:AYZ0103AGRLC, symbol SP3T
- removed U2: ROE-0505S, dcdc:ROE-DCDC, symbol ROE-0505S
Connections:
- net labels removed: +5VP, PWR_BR_IS, REGOUT, TPWR
- wire segments 238 -> 145

Commit message: finishing off
Parts:
- R1, R10, R11, R12, R13, R15, R2, R21, R22, R3, R4, R5, R6, R7, R8, R9: footprint Resistors_SMD:R_0603 -> passives-7351:C0603-N
- SW1, SW3: footprint Buttons_Switches_SMD:SW_SPST_EVQPE1 -> tactile_SPST:SW_SPST_EVQPE1
- Y1: footprint Crystals:Crystal_FOX-FE_SMD -> ABM7:ABM7
Changed lines of the file:
@@
 F 0 "R3" H 4030 3370 50  0000 L CNN
 F 1 "22" H 4030 3310 50  0000 L CNN
-F 2 "Resistors_SMD:R_0603" H 4000 3350 60  0001 C CNN
+F 2 "passives-7351:C0603-N" H 4000 3350 60  0001 C CNN
 F 3 "" H 4000 3350 60  0000 C CNN
 	1    4000 3350
@@
 F 0 "R4" H 4030 3470 50  0000 L CNN
 F 1 "22" H 4030 3410 50  0000 L CNN
-F 2 "Resistors_SMD:R_0603" H 4000 3450 60  0001 C CNN
+F 2 "passives-7351:C0603-N" H 4000 3450 60  0001 C CNN
 F 3 "" H 4000 3450 60  0000 C CNN
 	1    4000 3450
@@
 F 0 "SW1" H 3950 5260 50  0000 C CNN
 F 1 "SW_PUSH" H 3800 5070 50  0000 C CNN
-F 2 "Buttons_Switches_SMD:SW_SPST_EVQPE1" H 3800 5150 60  0001 C CNN
+F 2 "tactile_SPST:SW_SPST_EVQPE1" H 3800 5150 60  0001 C CNN
 F 3 "" H 3800 5150 60  0000 C CNN
 	1    3800 5150
@@
 F 0 "R1" H 3530 4970 50  0000 L CNN
 F 1 "10k" H 3530 4910 50  0000 L CNN
-F 2 "Resistors_SMD:R_0603" H 3500 4950 60  0001 C CNN
+F 2 "passives-7351:C0603-N" H 3500 4950 60  0001 C CNN
 F 3 "" H 3500 4950 60  0000 C CNN
 	1    3500 4950
@@
 F 0 "R2" H 4030 3070 50  0000 L CNN
 F 1 "1.5k" H 4030 3010 50  0000 L CNN
-F 2 "Resistors_SMD:R_0603" H 4000 3050 60  0001 C CNN
+F 2 "passives-7351:C0603-N" H 4000 3050 60  0001 C CNN
 F 3 "" H 4000 3050 60  0000 C CNN
 	1    4000 3050
@@
 F 0 "Y1" H 1150 4750 50  0000 C CNN
 F 1 "Crystal_Small" H 1150 4550 50  0000 C CNN
-F 2 "Crystals:Crystal_FOX-FE_SMD" H 1150 4650 60  0001 C CNN
+F 2 "ABM7:ABM7" H 1150 4650 60  0001 C CNN
 F 3 "" H 1150 4650 60  0000 C CNN
 	1    1150 4650
@@
 F 0 "R5" H 4630 5120 50  0000 L CNN
 F 1 "4.7k" H 4630 5060 50  0000 L CNN
-F 2 "Resistors_SMD:R_0603" H 4600 5100 60  0001 C CNN
+F 2 "passives-7351:C0603-N" H 4600 5100 60  0001 C CNN
 F 3 "" H 4600 5100 60  0000 C CNN
 	1    4600 5100
@@
 F 0 "R6" H 4630 5420 50  0000 L CNN
 F 1 "10k" H 4630 5360 50  0000 L CNN
-F 2 "Resistors_SMD:R_0603" H 4600 5400 60  0001 C CNN
+F 2 "passives-7351:C0603-N" H 4600 5400 60  0001 C CNN
 F 3 "" H 4600 5400 60  0000 C CNN
 	1    4600 5400
@@
 F 0 "R12" H 6080 2670 50  0000 L CNN
 F 1 "4.7k" H 6080 2610 50  0000 L CNN
-F 2 "Resistors_SMD:R_0603" H 6050 2650 60  0001 C CNN
+F 2 "passives-7351:C0603-N" H 6050 2650 60  0001 C CNN
 F 3 "" H 6050 2650 60  0000 C CNN
 	1    6050 2650
@@
 F 0 "R13" H 7580 2570 50  0000 L CNN
 F 1 "4.7k" H 7580 2510 50  0000 L CNN
-F 2 "Resistors_SMD:R_0603" H 7550 2550 60  0001 C CNN
+F 2 "passives-7351:C0603-N" H 7550 2550 60  0001 C CNN
 F 3 "" H 7550 2550 60  0000 C CNN
 	1    7550 2550
@@
 F 0 "R8" H 2880 6420 50  0000 L CNN
 F 1 "330" H 2880 6360 50  0000 L CNN
-F 2 "Resistors_SMD:R_0603" H 2850 6400 60  0001 C CNN
+F 2 "passives-7351:C0603-N" H 2850 6400 60  0001 C CNN
 F 3 "" H 2850 6400 60  0000 C CNN
 	1    2850 6400
@@
 F 0 "R9" H 2880 6720 50  0000 L CNN
 F 1 "330" H 2880 6660 50  0000 L CNN
-F 2 "Resistors_SMD:R_0603" H 2850 6700 60  0001 C CNN
+F 2 "passives-7351:C0603-N" H 2850 6700 60  0001 C CNN
 F 3 "" H 2850 6700 60  0000 C CNN
 	1    2850 6700
@@
 F 0 "R10" H 2880 7020 50  0000 L CNN
 F 1 "330" H 2880 6960 50  0000 L CNN
-F 2 "Resistors_SMD:R_0603" H 2850 7000 60  0001 C CNN
+F 2 "passives-7351:C0603-N" H 2850 7000 60  0001 C CNN
 F 3 "" H 2850 7000 60  0000 C CNN
 	1    2850 7000
@@
 F 0 "R11" H 2880 7320 50  0000 L CNN
 F 1 "330" H 2880 7260 50  0000 L CNN
-F 2 "Resistors_SMD:R_0603" H 2850 7300 60  0001 C CNN
+F 2 "passives-7351:C0603-N" H 2850 7300 60  0001 C CNN
 F 3 "" H 2850 7300 60  0000 C CNN
 	1    2850 7300
@@
 F 0 "R7" H 10830 3670 50  0000 L CNN
 F 1 "330" H 10830 3610 50  0000 L CNN
-F 2 "Resistors_SMD:R_0603" H 10800 3650 60  0001 C CNN
+F 2 "passives-7351:C0603-N" H 10800 3650 60  0001 C CNN
 F 3 "" H 10800 3650 60  0000 C CNN
 	1    10800 3650
@@
 F 0 "R15" H 1280 3020 50  0000 L CNN
 F 1 "10k" H 1280 2960 50  0000 L CNN
-F 2 "Resistors_SMD:R_0603" H 1250 3000 60  0001 C CNN
+F 2 "passives-7351:C0603-N" H 1250 3000 60  0001 C CNN
 F 3 "" H 1250 3000 60  0000 C CNN
 	1    1250 3000
@@
 F 0 "SW3" H 1100 2760 50  0000 C CNN
 F 1 "SW_PUSH" H 950 2570 50  0000 C CNN
-F 2 "Buttons_Switches_SMD:SW_SPST_EVQPE1" H 950 2650 60  0001 C CNN
+F 2 "tactile_SPST:SW_SPST_EVQPE1" H 950 2650 60  0001 C CNN
 F 3 "" H 950 2650 60  0000 C CNN
 	1    950  2650
@@
 F 0 "R21" H 5980 1620 50  0000 L CNN
 F 1 "4.7k" H 5980 1560 50  0000 L CNN
-F 2 "Resistors_SMD:R_0603" H 5950 1600 60  0001 C CNN
+F 2 "passives-7351:C0603-N" H 5950 1600 60  0001 C CNN
 F 3 "" H 5950 1600 60  0000 C CNN
 	1    5950 1600
@@
 F 0 "R22" H 7630 1420 50  0000 L CNN
 F 1 "4.7k" H 7630 1360 50  0000 L CNN
-F 2 "Resistors_SMD:R_0603" H 7600 1400 60  0001 C CNN
+F 2 "passives-7351:C0603-N" H 7600 1400 60  0001 C CNN
 F 3 "" H 7600 1400 60  0000 C CNN
 	1    7600 1400

Commit message: done
Parts:
- removed P3: TC2030-CTX, Tag-Connect:TC2030-NL_SMALL, symbol TC2030-CTX
- removed R21, R22: 4.7k, passives-7351:C0603-N, symbol R_Small
- J1: footprint Pin_Headers:Pin_Header_Straight_2x05_Pitch1.27mm -> agg:FTSH-105-01-L-DV-K
- P2: footprint Connectors_Molex:Connector_Molex_PicoBlade_53261-0471 -> agg:SM04B-PASS
- renumbered C18 to C10, C19 to C11, IC4 to IC2, R5 to R1, R15 to R10, R7 to R14, R8 to R2, R9 to R3, R10 to R4, R6 to R5, R1 to R6, R2 to R7, R3 to R8, R4 to R9, SW3 to SW1, SW1 to SW2
Connections:
- wire segments 145 -> 133
